File: docs/assets/pcb/light-v0.1/kicad/controller.kicad_sch (KiCad schematic)
At the start: 23 parts, among them J15 UART DEBUG, J17 ARM SWITCH, U1 ESP32-C6-WROOM-1-N8, U5 SN74LVC08APWR, U6 SN74LVC1G04DBVR

Commit message: Refresh PCB chapters from verified central LED snapshots
Parts:
- U5: value SN74LVC08APWR -> 74HCS08PWJ; symbol EL:SN74LVC08A -> EL:74HCS08; MPN SN74LVC08APWR -> 74HCS08PWJ; Manufacturer Texas Instruments -> Nexperia
Changed lines of the file:
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@@
           (size 1.0 1.0)))))
   (symbol
-    (lib_id "EL:SN74LVC08A")
+    (lib_id "EL:74HCS08")
     (at 121.92 238.76 0)
     (unit 1)
@@
         (font
           (size 1.0 1.0))))
-    (property "Value" "SN74LVC08APWR"
+    (property "Value" "74HCS08PWJ"
       (at 142.24 220.98 0.0)
       (effects
@@
         (font
           (size 1.0 1.0))))
-    (property "MPN" "SN74LVC08APWR"
+    (property "MPN" "74HCS08PWJ"
       (at 121.92 238.76 0.0)
       (hide yes)
@@
         (font
           (size 1.0 1.0))))
-    (property "Manufacturer" "Texas Instruments"
+    (property "Manufacturer" "Nexperia"
       (at 121.92 238.76 0.0)
       (hide yes)
@@
         (font
           (size 1.0 1.0))))
-    (property "Datasheet" "https://www.ti.com/lit/ds/symlink/sn74lvc08a.pdf"
+    (property "Datasheet" "https://assets.nexperia.com/documents/data-sheet/74HCS08.pdf"
       (at 121.92 238.76 0.0)
       (hide yes)
