File: docs/assets/pcb/light-v0.1/kicad/engineered-lighting-rev-a.kicad_pcb (KiCad board)
At the start: 8 copper layers, 76.2 x 75.1 mm, 269 parts, among them J1 24V INPUT, J10 SPOT 2, J11 SPOT 3, J12 MOTOR 1, J13 MOTOR 2, J14 USB DATA /24V REQUIRED, J15 UART DEBUG, J16 BRAKE / BUS, J17 ARM SWITCH, J18 GPIO EXPANSION 3V3, J2 ZONE 1, J3 ZONE 2, J4 ZONE 3, J5 ZONE 4, J6 ZONE 5, J7 ZONE 6, J8 ZONE 7, J9 SPOT 1, Q101 AO3422, Q102 AO3422, Q103 AO3422, Q104 AO3422, Q105 AO3422, Q106 AO3422, Q107 AO3422, Q108 AO3422, Q109 AO3422, Q110 AO3422, Q111 AO3422, Q112 AO3422, Q113 AO3422, Q114 AO3422, Q115 AO3422, Q116 AO3422, Q117 AO3422, Q118 AO3422, Q119 AO3422, Q120 AO3422, Q121 AO3422, Q30 MMBT3904, Q500 100V reverse blocking MOSFET, Q501 fast reverse gate pull-down, U1 ESP32-C6-WROOM-1-N8, U10 24V to 5V 1A buck, U11 5V to 3.3V 1A fixed buck, U12 24V input eFuse / 4.5A nominal, U13 switched ambient gate bias, U14 spot branch gated eFuse 0.494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, U15 ESDS302, U16 NUP2105LT1G, U17 TMUXHS221F, U18 TPS3808G33, U19 SN74LVC1G97 AND Schmitt, U2 PCA9685PW,118, U20 TMP112AIDRLR, U3 PCA9685PW,118, U4 TCAN1042HGVDRQ1, U5 SN74LVC08APWR, U500 27V flat-clamp transient prot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, U501 27V flat-clamp transient prot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, U6 SN74LVC1G04DBVR, U7 333mA spotlight CC driver, U8 333mA spotlight CC driver, U9 333mA spotlight CC driver

Commit message: Refresh PCB chapters from verified central LED snapshots
Parts:
- removed J3: ZONE 2, Connector_JST:JST_GH_SM04B-GHS-TB_1x04-1MP_P1.25mm_Horizontal
- removed J4: ZONE 3, Connector_JST:JST_GH_SM04B-GHS-TB_1x04-1MP_P1.25mm_Horizontal
- removed J5: ZONE 4, ELF:Enclosure_J5
- removed J6: ZONE 5, ELF:Enclosure_J6
- removed J7: ZONE 6, Connector_JST:JST_GH_SM04B-GHS-TB_1x04-1MP_P1.25mm_Horizontal
- J2: value ZONE 1 -> 2005280300 / 6-ZONE FLEX; footprint Connector_JST:JST_GH_SM04B-GHS-TB_1x04-1MP_P1.25mm_Horizontal -> ELF:Molex_2005280300_30P_Central_LED
- R206: moved to F.Cu
- R526, R527, R528: value 10k -> 910
- U5: value SN74LVC08APWR -> 74HCS08PWJ
- moved J2 13.6 mm to (70.0, 99.4), turned to -90 degrees
- moved R206 11.6 mm to (76.6, 101.8)
- moved Q106 1.00 mm to (74.0, 97.5)
- moved R106 0.79 mm to (73.8, 101.2)
Connections:
- J2 pad 1: ZONE1_24V -> ZONE4_24V
- J2 pad 2: ZONE1_W -> ZONE4_24V
- J2 pad 3: ZONE1_N -> ZONE4_W
- J2 pad 4: ZONE1_C -> ZONE4_N
Routing:
- net ZONE6_W: track 18.8 -> 161.3 mm, vias 2 -> 8
- net ZONE6_N: track 20.1 -> 143.3 mm, vias 2 -> 7
- net ZONE6_C: track 9.23 -> 117.9 mm, vias 2 -> 8
- net ZONE6_24V: track 39.7 -> 135.3 mm, vias 4 -> 5
- net ZONE5_24V: track 33.7 -> 118.8 mm, vias 6 -> 11
- net ZONE5_C: track 18.3 -> 102.4 mm, vias 2 -> 12
- net ZONE4_C: track 19.0 -> 89.2 mm, vias 2 -> 6
- net ZONE5_W: track 22.1 -> 90.9 mm, vias 2 -> 10
- net ZONE5_N: track 12.7 -> 73.2 mm, vias 0 -> 8
- net ZONE1_C: track 34.1 -> 94.4 mm, vias 4 -> 8
- net PWM_03: track 47.2 -> 106.2 mm, vias 3 -> 10
- net ZONE1_W: track 20.0 -> 76.8 mm, vias 2 -> 6
- net ZONE3_24V: track 51.2 -> 105.7 mm, vias 4 -> 7
- net PWM_06: track 37.0 -> 82.1 mm, vias 2 -> 4
- net SPOT3_CTRL: track 74.2 -> 39.3 mm, vias 9 -> 2
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Other:
- board text added: "30"
- board text added: "ENGINEERED LIGHTING LIGHT v0.2"
- board text added: "J2 LED Z1-6"
- board text removed: "ENGINEERED LIGHTING LIGHT v0.1"
- board text removed: "J2 Z1"
- board text removed: "J3 Z2"
- board text removed: "J4 Z3"
- board text removed: "J5 Z4"
- board text removed: "J6 Z5"
- board text removed: "J7 Z6"
