File: docs/assets/pcb/light-v0.1/kicad/engineered-lighting-rev-a.kicad_pcb (KiCad board)
At the start: 8 copper layers, 76.2 x 75.1 mm, 264 parts, among them J1 24V INPUT, J10 SPOT 2, J11 SPOT 3, J12 MOTOR 1, J13 MOTOR 2, J14 USB DATA /24V REQUIRED, J15 UART DEBUG, J16 BRAKE / BUS, J17 ARM SWITCH, J18 GPIO EXPANSION 3V3, J2 2005280300 / 6-ZONE FLEX, J8 ZONE 7, J9 SPOT 1, Q101 AO3422, Q102 AO3422, Q103 AO3422, Q104 AO3422, Q105 AO3422, Q106 AO3422, Q107 AO3422, Q108 AO3422, Q109 AO3422, Q110 AO3422, Q111 AO3422, Q112 AO3422, Q113 AO3422, Q114 AO3422, Q115 AO3422, Q116 AO3422, Q117 AO3422, Q118 AO3422, Q119 AO3422, Q120 AO3422, Q121 AO3422, Q30 MMBT3904, Q500 100V reverse blocking MOSFET, Q501 fast reverse gate pull-down, U1 ESP32-C6-WROOM-1-N8, U10 24V to 5V 1A buck, U11 5V to 3.3V 1A fixed buck, U12 24V input eFuse / 4.5A nominal, U13 switched ambient gate bias, U14 spot branch gated eFuse 0.494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, U15 ESDS302, U16 NUP2105LT1G, U17 TMUXHS221F, U18 TPS3808G33, U19 SN74LVC1G97 AND Schmitt, U2 PCA9685PW,118, U20 TMP112AIDRLR, U3 PCA9685PW,118, U4 TCAN1042HGVDRQ1, U5 74HCS08PWJ, U500 27V flat-clamp transient prot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, U501 27V flat-clamp transient prot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, U6 SN74LVC1G04DBVR, U7 333mA spotlight CC driver, U8 333mA spotlight CC driver, U9 333mA spotlight CC driver

Commit message: Refresh PCB chapters for grouped arm connectors and branded revision
Parts:
- removed J10: SPOT 2, ELF:Enclosure_J10
- removed J11: SPOT 3, Connector_JST:JST_GH_BM02B-GHS-TBT_1x02-1MP_P1.25mm_Vertical
- J9: value SPOT 1 -> SPOTLIGHT 3 PAIRS; footprint ELF:Enclosure_J9 -> EL:JST_GH_BM06B-GHS-TBT_1x06-1MP_P1.25mm_Vertical
- moved J9 65.5 mm to (127.0, 116.0), turned to 180 degrees
Routing:
- net SPOT1_LED_MINUS: track 33.2 -> 112.6 mm, vias 2 -> 5
- net SPOT3_LED_PLUS: track 25.6 -> 104.1 mm, vias 4 -> 7
- net SPOT1_LED_PLUS: track 23.8 -> 93.0 mm, vias 4 -> 7
- net SPOT3_LED_MINUS: track 11.7 -> 78.8 mm, vias 0 -> 2
- net SPOT2_LED_MINUS: track 55.4 -> 92.1 mm, vias 4 -> 6
- net SPOT2_LED_PLUS: track 38.7 -> 73.4 mm, vias 4 -> 6
- net USB_SENSE_BASE: track 77.8 -> 81.3 mm, vias 5 -> 7
- net ZONE6_C: track 117.9 -> 118.9 mm, vias 8 -> 9
Other:
- board text added: ""A room is not a room"
- board text added: "J9 SPOT"
- board text added: "LIGHT v0.2"
- board text added: "engineered lighting"
- board text added: "engineered.lighting"
- board text added: "without natural light.""
- board text added: "— Louis Kahn"
- board text removed: "ENGINEERED LIGHTING LIGHT v0.2"
- board text removed: "J10 S2"
- board text removed: "J11 S3"
- board text removed: "J9 S1"
