File: docs/assets/pcb/light-v0.1/kicad/engineered-lighting-rev-a.kicad_sch (KiCad schematic)
At the start: 0 parts

Commit message: Refresh PCB chapters from verified central LED snapshots
Other:
- added sheet central_led_interface (central_led_interface.kicad_sch)
Changed lines of the file:
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@@
   (title_block
     (title "Integrated lighting controller")
-    (date "2026-09-06")
-    (rev "A draft")
+    (date "2026-09-08")
+    (rev "LIGHT v0.2 candidate")
     (company "Engineered Lighting")
     (comment 1 "ENGINEERING DRAFT - see release status before fabrication"))
@@
     (path "/"
       (page "1")))
-  (embedded_fonts no))
+  (embedded_fonts no)
+  (sheet
+    (at 213.36 255.27)
+    (size 81.28 13.97)
+    (stroke
+      (width 0)
+      (type default))
+    (fill
+      (color 0 0 0 0))
+    (property "Sheetname" "central_led_interface"
+      (at 213.36 254.0 0.0)
+      (effects
+        (font
+          (size 1.0 1.0))))
+    (property "Sheetfile" "central_led_interface.kicad_sch"
+      (at 213.36 270.51 0.0)
+      (effects
+        (font
+          (size 1.0 1.0))))
+    (instances
+      (project "engineered-lighting-rev-a"
+        (path "/964013ac-cca6-5de7-b648-d598a25a58e0"
+          (page "20"))))))
