File: docs/assets/pcb/light-v0.1/kicad/power_1.kicad_sch (KiCad schematic)
At the start: 31 parts, among them Q500 100V reverse blocking MOSFET, Q501 fast reverse gate pull-down, U12 24V input eFuse / 4.5A nominal

Commit message: Refresh PCB chapters from verified central LED snapshots
Parts:
- C500, C502, C503, C505: Manufacturer (none) -> Murata
- C501: Manufacturer (none) -> TDK
- C504: Manufacturer (none) -> Cornell Dubilier / Knowles
- D500, F1, F10, F11, F2, F3, F4, F5, F6, F7, F8, F9: Manufacturer (none) -> Littelfuse
- Q501: Manufacturer (none) -> Nexperia
- R500, R501, R502, R503, R504, R505, R506, R507, R508, R509: Manufacturer (none) -> Yageo
Changed lines of the file:
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@@
         (font
           (size 1.0 1.0))))
-    (property "Manufacturer" ""
+    (property "Manufacturer" "Nexperia"
       (at 116.84 119.38 0.0)
       (hide yes)
@@
         (font
           (size 1.0 1.0))))
-    (property "Manufacturer" ""
+    (property "Manufacturer" "Littelfuse"
       (at 30.48 152.4 0.0)
       (hide yes)
@@
         (font
           (size 1.0 1.0))))
-    (property "Manufacturer" ""
+    (property "Manufacturer" "Littelfuse"
       (at 35.56 66.04 0.0)
       (hide yes)
@@
         (font
           (size 1.0 1.0))))
-    (property "Manufacturer" ""
+    (property "Manufacturer" "Littelfuse"
       (at 35.56 229.87 0.0)
       (hide yes)
@@
         (font
           (size 1.0 1.0))))
-    (property "Manufacturer" ""
+    (property "Manufacturer" "Littelfuse"
       (at 106.68 229.87 0.0)
       (hide yes)
@@
         (font
           (size 1.0 1.0))))
-    (property "Manufacturer" ""
+    (property "Manufacturer" "Littelfuse"
       (at 177.8 229.87 0.0)
       (hide yes)
@@
         (font
           (size 1.0 1.0))))
-    (property "Manufacturer" ""
+    (property "Manufacturer" "Littelfuse"
       (at 248.92 229.87 0.0)
       (hide yes)
@@
         (font
           (size 1.0 1.0))))
-    (property "Manufacturer" ""
+    (property "Manufacturer" "Littelfuse"
       (at 320.04 229.87 0.0)
       (hide yes)
@@
         (font
           (size 1.0 1.0))))
-    (property "Manufacturer" ""
+    (property "Manufacturer" "Littelfuse"
       (at 35.56 248.92 0.0)
       (hide yes)
@@
         (font
           (size 1.0 1.0))))
-    (property "Manufacturer" ""
+    (property "Manufacturer" "Littelfuse"
       (at 106.68 248.92 0.0)
       (hide yes)
@@
         (font
           (size 1.0 1.0))))
-    (property "Manufacturer" ""
+    (property "Manufacturer" "Littelfuse"
       (at 177.8 248.92 0.0)
       (hide yes)
@@
         (font
           (size 1.0 1.0))))
-    (property "Manufacturer" ""
+    (property "Manufacturer" "Littelfuse"
       (at 248.92 248.92 0.0)
       (hide yes)
@@
         (font
           (size 1.0 1.0))))
-    (property "Manufacturer" ""
+    (property "Manufacturer" "Littelfuse"
       (at 320.04 248.92 0.0)
       (hide yes)
@@
         (font
           (size 1.0 1.0))))
-    (property "Manufacturer" ""
+    (property "Manufacturer" "Yageo"
       (at 78.74 152.4 0.0)
       (hide yes)
@@
         (font
           (size 1.0 1.0))))
-    (property "Manufacturer" ""
+    (property "Manufacturer" "Yageo"
       (at 127.0 152.4 0.0)
       (hide yes)
@@
         (font
           (size 1.0 1.0))))
-    (property "Manufacturer" ""
+    (property "Manufacturer" "Yageo"
       (at 175.26 152.4 0.0)
       (hide yes)
@@
         (font
           (size 1.0 1.0))))
-    (property "Manufacturer" ""
+    (property "Manufacturer" "Yageo"
       (at 223.52 152.4 0.0)
       (hide yes)
@@
         (font
           (size 1.0 1.0))))
-    (property "Manufacturer" ""
+    (property "Manufacturer" "Yageo"
       (at 271.78 152.4 0.0)
       (hide yes)
@@
         (font
           (size 1.0 1.0))))
-    (property "Manufacturer" ""
+    (property "Manufacturer" "Yageo"
       (at 320.04 152.4 0.0)
       (hide yes)
@@
         (font
           (size 1.0 1.0))))
-    (property "Manufacturer" ""
+    (property "Manufacturer" "Yageo"
       (at 368.3 152.4 0.0)
       (hide yes)
@@
         (font
           (size 1.0 1.0))))
-    (property "Manufacturer" ""
+    (property "Manufacturer" "Yageo"
       (at 30.48 195.58 0.0)
       (hide yes)
@@
         (font
           (size 1.0 1.0))))
-    (property "Manufacturer" ""
+    (property "Manufacturer" "Yageo"
       (at 78.74 195.58 0.0)
       (hide yes)
@@
         (font
           (size 1.0 1.0))))
-    (property "Manufacturer" ""
+    (property "Manufacturer" "Yageo"
       (at 127.0 195.58 0.0)
       (hide yes)
@@
         (font
           (size 1.0 1.0))))
-    (property "Manufacturer" ""
+    (property "Manufacturer" "Murata"
       (at 175.26 195.58 0.0)
       (hide yes)
@@
         (font
           (size 1.0 1.0))))
-    (property "Manufacturer" ""
+    (property "Manufacturer" "TDK"
       (at 223.52 195.58 0.0)
       (hide yes)
@@
         (font
           (size 1.0 1.0))))
-    (property "Manufacturer" ""
+    (property "Manufacturer" "Murata"
       (at 271.78 195.58 0.0)
       (hide yes)
@@
         (font
           (size 1.0 1.0))))
-    (property "Manufacturer" ""
+    (property "Manufacturer" "Murata"
       (at 320.04 195.58 0.0)
       (hide yes)
@@
         (font
           (size 1.0 1.0))))
-    (property "Manufacturer" ""
+    (property "Manufacturer" "Cornell Dubilier / Knowles"
       (at 353.06 71.12 0.0)
       (hide yes)
@@
         (font
           (size 1.0 1.0))))
-    (property "Manufacturer" ""
+    (property "Manufacturer" "Murata"
       (at 368.3 195.58 0.0)
       (hide yes)
