File: docs/assets/pcb/light-v0.1/kicad/power_2.kicad_sch (KiCad schematic)
At the start: 24 parts, among them J1 24V INPUT, J16 BRAKE / BUS, U10 24V to 5V 1A buck, U11 5V to 3.3V 1A fixed buck, U13 switched ambient gate bias, U501 27V flat-clamp transient prot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

Commit message: Refresh PCB chapters from verified central LED snapshots
Parts:
- C506, C509, C510, C511, C513, C514, C515: Manufacturer (none) -> Murata
- C507, C508: Manufacturer (none) -> TDK
- D505: Manufacturer (none) -> Diodes Incorporated
- L500, L501: Manufacturer (none) -> Bourns
- R510, R511, R512, R513: Manufacturer (none) -> Yageo
Changed lines of the file:
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@@
         (font
           (size 1.0 1.0))))
-    (property "Manufacturer" ""
+    (property "Manufacturer" "Bourns"
       (at 144.78 73.66 0.0)
       (hide yes)
@@
         (font
           (size 1.0 1.0))))
-    (property "Manufacturer" ""
+    (property "Manufacturer" "Murata"
       (at 35.56 71.12 0.0)
       (hide yes)
@@
         (font
           (size 1.0 1.0))))
-    (property "Manufacturer" ""
+    (property "Manufacturer" "TDK"
       (at 121.92 43.18 0.0)
       (hide yes)
@@
         (font
           (size 1.0 1.0))))
-    (property "Manufacturer" ""
+    (property "Manufacturer" "TDK"
       (at 43.18 111.76 0.0)
       (hide yes)
@@
         (font
           (size 1.0 1.0))))
-    (property "Manufacturer" ""
+    (property "Manufacturer" "Murata"
       (at 68.58 111.76 0.0)
       (hide yes)
@@
         (font
           (size 1.0 1.0))))
-    (property "Manufacturer" ""
+    (property "Manufacturer" "Murata"
       (at 177.8 96.52 0.0)
       (hide yes)
@@
         (font
           (size 1.0 1.0))))
-    (property "Manufacturer" ""
+    (property "Manufacturer" "Murata"
       (at 203.2 96.52 0.0)
       (hide yes)
@@
         (font
           (size 1.0 1.0))))
-    (property "Manufacturer" ""
+    (property "Manufacturer" "Yageo"
       (at 154.94 137.16 0.0)
       (hide yes)
@@
         (font
           (size 1.0 1.0))))
-    (property "Manufacturer" ""
+    (property "Manufacturer" "Yageo"
       (at 154.94 167.64 0.0)
       (hide yes)
@@
         (font
           (size 1.0 1.0))))
-    (property "Manufacturer" ""
+    (property "Manufacturer" "Yageo"
       (at 35.56 149.86 0.0)
       (hide yes)
@@
         (font
           (size 1.0 1.0))))
-    (property "Manufacturer" ""
+    (property "Manufacturer" "Bourns"
       (at 342.9 68.58 0.0)
       (hide yes)
@@
         (font
           (size 1.0 1.0))))
-    (property "Manufacturer" ""
+    (property "Manufacturer" "Murata"
       (at 375.92 99.06 0.0)
       (hide yes)
@@
         (font
           (size 1.0 1.0))))
-    (property "Manufacturer" ""
+    (property "Manufacturer" "Yageo"
       (at 241.3 137.16 0.0)
       (hide yes)
@@
         (font
           (size 1.0 1.0))))
-    (property "Manufacturer" ""
+    (property "Manufacturer" "Murata"
       (at 68.58 205.74 0.0)
       (hide yes)
@@
         (font
           (size 1.0 1.0))))
-    (property "Manufacturer" ""
+    (property "Manufacturer" "Murata"
       (at 180.34 205.74 0.0)
       (hide yes)
@@
         (font
           (size 1.0 1.0))))
-    (property "Manufacturer" ""
+    (property "Manufacturer" "Diodes Incorporated"
       (at 246.38 228.6 0.0)
       (hide yes)
